File: pcb/stm32_expansion/stm32_expansion.sch (KiCad schematic (older format))
At the start: 8 parts, among them J1 Conn_01x02_Male, P1 Conn_02x11_Odd_Even, P2 Conn_02x11_Odd_Even, P3 Conn_02x11_Odd_Even, P4 Conn_02x11_Odd_Even, P5 Conn_01x20_Female, P6 Conn_01x20_Female, U1 TJA1051T

Commit message: Update schematic.
Connections:
- net Pin01: now also P6.16 (Pin_16)
- net Pin02: now also P6.15 (Pin_15)
- net Pin03: now also P6.14 (Pin_14)
- net Pin04: now also P6.13 (Pin_13)
- net Pin05: now also P6.11 (Pin_11)
- net Pin06: now also P6.10 (Pin_10)
- net Pin07: now also P5.15 (Pin_15)
- net Pin08: now also P5.16 (Pin_16)
- net Pin14: now also P6.9 (Pin_9)
- net Pin15: now also P6.8 (Pin_8)
- net Pin16: now also P5.13 (Pin_13)
- net Pin17: now also P5.14 (Pin_14)
- net Pin30: no longer P6.8 (Pin_8)
- net Pin33: no longer P6.9 (Pin_9)
- net Pin34: no longer P6.10 (Pin_10)
- net Pin35: no longer P6.11 (Pin_11)
- net Pin37: no longer P6.13 (Pin_13)
- net Pin38: no longer P6.14 (Pin_14)
- net Pin39: no longer P6.15 (Pin_15)
- net Pin40: no longer P6.16 (Pin_16)
Other:
- note added: "A10 (TIM1_CH3)"
- note added: "A11 (TIM1_CH4)"
- note added: "A15 (TIM2_CH1)"
- note added: "A8 (TIM1_CH1)"
- note added: "A9 (TIM1_CH2)"
- note added: "B0 (TIM3_CH3)"
- note added: "B1 (TIM3_CH4)"
- note added: "B10 (TIM2_CH3)"
- note added: "B11 (TIM2_CH4)"
- note added: "B3 (TIM2_CH2)"
- note added: "B4 (TIM3_CH1)"
- note added: "B5 (TIM3_CH2)"
- note removed: "A10"
- note removed: "A11"
- note removed: "A15"
- note removed: "A8"
- note removed: "A9"
- note removed: "B0"
- note removed: "B1"
- note removed: "B10"
- note removed: "B11"
- note removed: "B3"
- note removed: "B4"
- note removed: "B5"
Changed lines of the file:
@@
 A7
 Text Notes 1300 4300 0    50   ~ 0
-B0
+B0 (TIM3_CH3)
 Text Notes 1300 4400 0    50   ~ 0
-B1
+B1 (TIM3_CH4)
 Text Notes 1300 4500 0    50   ~ 0
-B10
+B10 (TIM2_CH3)
 Text Notes 1300 4600 0    50   ~ 0
-B11
+B11 (TIM2_CH4)
 Text Notes 1300 4700 0    50   ~ 0
 R
@@
 B6
 Text Notes 2950 3800 0    50   ~ 0
-B5
+B5 (TIM3_CH2)
 Text Notes 2950 3900 0    50   ~ 0
-B4
+B4 (TIM3_CH1)
 Text Notes 2950 4000 0    50   ~ 0
-B3
+B3 (TIM2_CH2)
 Text Notes 2950 4100 0    50   ~ 0
-A15
+A15 (TIM2_CH1)
 Text Notes 2950 4200 0    50   ~ 0
 A12
 Text Notes 2950 4300 0    50   ~ 0
-A11
+A11 (TIM1_CH4)
 Text Notes 2950 4400 0    50   ~ 0
-A10
+A10 (TIM1_CH3)
 Text Notes 2950 4500 0    50   ~ 0
-A9
+A9 (TIM1_CH2)
 Text Notes 2950 4600 0    50   ~ 0
-A8
+A8 (TIM1_CH1)
 Text Notes 2950 4700 0    50   ~ 0
 B15
@@
 Pin29
 Text Label 2450 3800 0    50   ~ 0
-Pin30
+Pin15
 Text Label 2450 3900 0    50   ~ 0
-Pin33
+Pin14
 Text Label 2450 4000 0    50   ~ 0
-Pin34
+Pin06
 Text Label 2450 4100 0    50   ~ 0
-Pin35
+Pin05
 Text Label 2450 4200 0    50   ~ 0
 Pin36
 Text Label 2450 4300 0    50   ~ 0
-Pin37
+Pin04
 Text Label 2450 4400 0    50   ~ 0
-Pin38
+Pin03
 Text Label 2450 4500 0    50   ~ 0
-Pin39
+Pin02
 Text Label 2450 4600 0    50   ~ 0
-Pin40
+Pin01
 Text Label 2450 4700 0    50   ~ 0
 Pin41
@@
 Text Label 2500 3300 0    50   ~ 0
 5V
+Text Label 800  4500 0    50   ~ 0
+Pin07
+Text Label 800  4600 0    50   ~ 0
+Pin08
+Text Label 800  4300 0    50   ~ 0
+Pin16
+Text Label 800  4400 0    50   ~ 0
+Pin17
+Wire Wire Line
+	800  4300 1050 4300
+Wire Wire Line
+	800  4400 1050 4400
+Wire Wire Line
+	800  4500 1050 4500
+Wire Wire Line
+	800  4600 1050 4600
 $EndSCHEMATC

Commit message: Update pcb.
Connections:
- net Pin18: now also P6.20 (Pin_20)
- net Pin19: now also P6.19 (Pin_19)
- net Pin20: now also P6.18 (Pin_18)
- net Pin21: now also P6.17 (Pin_17)
- net Pin26: no longer P6.4 (Pin_4)
- net Pin27: no longer P6.5 (Pin_5)
- net Pin28: no longer P6.6 (Pin_6)
- net Pin29: no longer P6.7 (Pin_7)
- net Pin36: no longer P6.12 (Pin_12)
- net Pin41: no longer P6.17 (Pin_17)
- net Pin42: no longer P6.18 (Pin_18)
- net Pin43: no longer P6.19 (Pin_19)
- net Pin44: no longer P6.20 (Pin_20)
Changed lines of the file:
@@
 Wire Wire Line
 	900  1950 1150 1950
-Text Label 2450 3400 0    50   ~ 0
-Pin26
-Text Label 2450 3500 0    50   ~ 0
-Pin27
-Text Label 2450 3600 0    50   ~ 0
-Pin28
-Text Label 2450 3700 0    50   ~ 0
-Pin29
 Text Label 2450 3800 0    50   ~ 0
 Pin15
@@
 Text Label 2450 4100 0    50   ~ 0
 Pin05
-Text Label 2450 4200 0    50   ~ 0
-Pin36
 Text Label 2450 4300 0    50   ~ 0
 Pin04
@@
 Pin01
 Text Label 2450 4700 0    50   ~ 0
-Pin41
+Pin21
 Text Label 2450 4800 0    50   ~ 0
-Pin42
+Pin20
 Text Label 2450 4900 0    50   ~ 0
-Pin43
+Pin19
 Text Label 2450 5000 0    50   ~ 0
-Pin44
-Wire Wire Line
-	2450 3400 2700 3400
-Wire Wire Line
-	2450 3500 2700 3500
-Wire Wire Line
-	2450 3600 2700 3600
-Wire Wire Line
-	2450 3700 2700 3700
+Pin18
 Wire Wire Line
 	2450 3800 2700 3800
@@
 	2450 4100 2700 4100
 Wire Wire Line
-	2450 4200 2700 4200
-Wire Wire Line
 	2450 4300 2700 4300

Commit message: Update pcb layout.
Parts:
- added C1: 0.1uF, Capacitor_Tantalum_SMD:CP_EIA-2012-12_Kemet-R, symbol Device:C
- added C2, C3: 30pF, Capacitor_Tantalum_SMD:CP_EIA-2012-12_Kemet-R, symbol Device:C
- added CAN1, UART1: Conn_01x04, Connector_PinSocket_2.54mm:PinSocket_1x04_P2.54mm_Vertical, symbol Connector_Generic:Conn_01x04
- added Can2: Conn_01x02, Connector_PinSocket_2.54mm:PinSocket_1x02_P2.54mm_Vertical, symbol Connector_Generic:Conn_01x02
- added M1, M2, M3: Conn_01x05, Connector_PinSocket_2.54mm:PinSocket_1x05_P2.54mm_Vertical, symbol Connector_Generic:Conn_01x05
- added R1, R2: 0R, Resistor_SMD:R_0805_2012Metric, symbol Device:R_US
- added R3: 120R, Resistor_SMD:R_0805_2012Metric, symbol Device:R_US
- added S1, S2, S3, S4, S5, S6: Conn_01x03, Connector_PinSocket_2.54mm:PinSocket_1x03_P2.54mm_Vertical, symbol Connector_Generic:Conn_01x03
Connections:
- net 5V: now also U1.3 (VCC), C1.1, CAN1.1 (Pin_1), S1.2 (Pin_2), S2.2 (Pin_2), S3.2 (Pin_2), S4.2 (Pin_2), S5.2 (Pin_2), S6.2 (Pin_2), UART1.2 (Pin_2)
- net GND: now also U1.2 (GND), U1.8 (S), C1.2, C2.2, C3.2, CAN1.4 (Pin_4), M1.1 (Pin_1), M2.1 (Pin_1), M3.1 (Pin_1), S1.1 (Pin_1), S2.1 (Pin_1), S3.1 (Pin_1), S4.1 (Pin_1), S5.1 (Pin_1), S6.1 (Pin_1), UART1.1 (Pin_1)
- net Pin76: now also M1.2 (Pin_2)
- net Pin77: now also M1.3 (Pin_3)
- net Pin78: now also M1.4 (Pin_4)
- net Pin81: now also M1.5 (Pin_5)
- net Pin82: now also M2.2 (Pin_2)
- net Pin83: now also M2.3 (Pin_3)
- net Pin84: now also M2.4 (Pin_4)
- net Pin85: now also M2.5 (Pin_5)
- net Pin86: now also M3.2 (Pin_2)
- net Pin87: now also M3.3 (Pin_3)
- net Pin88: now also M3.4 (Pin_4)
- net Pin89: now also M3.5 (Pin_5)
- net Pin90: now also S1.3 (Pin_3)
- net Pin91: now also S2.3 (Pin_3)
- net Pin92: now also S3.3 (Pin_3)
- net Pin95: now also S4.3 (Pin_3)
- net Pin96: now also S5.3 (Pin_3)
- net Pin97: now also S6.3 (Pin_3)
- net UART2_TX: now reaches P5.7 (Pin_7)
- net UART2_TX: now also UART1.3 (Pin_3)
- net UART2_RX: now reaches P5.8 (Pin_8)
- net UART2_RX: now also UART1.4 (Pin_4)
- net CAN_TX: now reaches P6.4 (Pin_4)
- net CAN_TX: now also U1.1 (TXD), CAN1.2 (Pin_2)
- net CAN_RX: now reaches P6.5 (Pin_5)
- net CAN_RX: now also U1.4 (RXD), CAN1.3 (Pin_3)
- net at U1.6 (CANL): now also R2.2
- net at U1.7 (CANH): now also R1.2
- new net: C2.1, Can2.1 (Pin_1), R1.1, R3.2
- new net: C3.1, Can2.2 (Pin_2), R2.1, R3.1

Commit message: update uart to lora.
Parts:
- removed UART1: Conn_01x04, Connector_PinSocket_2.54mm:PinSocket_1x04_P2.54mm_Vertical, symbol Connector_Generic:Conn_01x04
- added LoRa1: Conn_01x07, Connector_PinSocket_2.54mm:PinSocket_1x07_P2.54mm_Vertical, symbol Connector_Generic:Conn_01x07
Connections:
- net 5V: now also LoRa1.2 (Pin_2)
- net GND: now also LoRa1.1 (Pin_1)
- net UART2_RX: now also LoRa1.4 (Pin_4)
- net UART2_TX: now also LoRa1.5 (Pin_5)
- net AUX: now reaches P5.4 (Pin_4)
- net AUX: now also LoRa1.3 (Pin_3)
- net MD0: now reaches P5.5 (Pin_5)
- net MD0: now also LoRa1.7 (Pin_7)
- net MD1: now reaches P5.6 (Pin_6)
- net MD1: now also LoRa1.6 (Pin_6)
Changed lines of the file:
@@
 Wire Wire Line
 	8550 3500 8850 3500
-$Comp
-L Connector_Generic:Conn_01x04 UART1
-U 1 1 61271737
-P 7650 5200
-F 0 "UART1" H 7730 5146 50  0000 L CNN
-F 1 "Conn_01x04" H 7730 5101 50  0001 L CNN
-F 2 "Connector_PinSocket_2.54mm:PinSocket_1x04_P2.54mm_Vertical" H 7650 5200 50  0001 C CNN
-F 3 "~" H 7650 5200 50  0001 C CNN
-	1    7650 5200
-	1    0    0    -1
-$EndComp
-Text Label 7250 5100 0    50   ~ 0
-GND
-Text Label 7250 5200 0    50   ~ 0
-5V
-Wire Wire Line
-	7250 5100 7450 5100
-Wire Wire Line
-	7250 5200 7450 5200
 Text Label 650  3700 0    50   ~ 0
 UART2_TX
@@
 Wire Wire Line
 	650  3800 1050 3800
-Text Label 7050 5300 0    50   ~ 0
-UART2_TX
-Text Label 7050 5400 0    50   ~ 0
-UART2_RX
-Wire Wire Line
-	7050 5300 7450 5300
-Wire Wire Line
-	7050 5400 7450 5400
 Text Label 2350 3400 0    50   ~ 0
 CAN_TX
@@
 Wire Wire Line
 	4550 6150 5050 6150
+$Comp
+L Connector_Generic:Conn_01x07 LoRa1
+U 1 1 611397ED
+P 7650 5350
+F 0 "LoRa1" H 7730 5346 50  0000 L CNN
+F 1 "Conn_01x07" H 7730 5301 50  0001 L CNN
+F 2 "Connector_PinSocket_2.54mm:PinSocket_1x07_P2.54mm_Vertical" H 7650 5350 50  0001 C CNN
+F 3 "~" H 7650 5350 50  0001 C CNN
+	1    7650 5350
+	1    0    0    -1
+$EndComp
+Text Label 7250 5050 0    50   ~ 0
+GND
+Text Label 7250 5150 0    50   ~ 0
+5V
+Text Label 7250 5250 0    50   ~ 0
+AUX
+Text Label 7050 5350 0    50   ~ 0
+UART2_RX
+Text Label 7050 5450 0    50   ~ 0
+UART2_TX
+Text Label 7250 5550 0    50   ~ 0
+MD1
+Text Label 7250 5650 0    50   ~ 0
+MD0
+Wire Wire Line
+	7250 5050 7450 5050
+Wire Wire Line
+	7250 5150 7450 5150
+Wire Wire Line
+	7250 5250 7450 5250
+Wire Wire Line
+	7050 5350 7450 5350
+Wire Wire Line
+	7050 5450 7450 5450
+Wire Wire Line
+	7250 5550 7450 5550
+Wire Wire Line
+	7250 5650 7450 5650
+Text Label 850  3500 0    50   ~ 0
+MD0
+Text Label 850  3600 0    50   ~ 0
+MD1
+Wire Wire Line
+	850  3500 1050 3500
+Wire Wire Line
+	850  3600 1050 3600
+Text Label 850  3400 0    50   ~ 0
+AUX
+Wire Wire Line
+	850  3400 1050 3400
 $EndSCHEMATC
